File: pcb/kicad/guitar.kicad_sch (KiCad schematic)
At the start: 34 parts, among them J5 Guitar in, Q1 BC857, U10 LM393, U9 OPA1642AIDR

Commit message: Pedalboard PCB: simulations A1-A8 and the values they changed
ngspice simulations of the guitar input, clip LED, ADC input, outputs,
headphones and the 12 V supply, read from the KiCad netlist and run with
TI's models (fetched by get-models.sh, not in git). All eight pass.

From the simulations: guitar RF filter 100 pF -> 22 pF, clip LED hold
100 nF / 2.2M / 1M with the LM393B, main output capacitors 47 uF.
The power-off thump when the lead is pulled is accepted for now
(sim/README.md).

Co-Authored-By: Claude Opus 5.5 <noreply@anthropic.com>
Parts:
- C43: value 100pF C0G -> 22pF C0G; Note RF filter at the op-amp pin -> RF filter at the op-amp pin: 7 MHz with the 1k. Small, beca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
- C51: value 2.2uF 25V -> 100nF; footprint Capacitor_SMD:CP_Elec_4x5.4 -> Capacitor_SMD:C_0603_1608Metric; symbol Device:C_Polarized -> Device:C; Note Hold: LED stays on about 100 ms after a peak (simulation A4) -> Hold: one 1 kHz peak 0.5 dB over the threshold lights the L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
- R44: Note Discharges the hold capacitor quickly (about 5 mA) -> Discharges the hold capacitor quickly: 5.5 mA, inside the L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
- R45: value 47k -> 2.2M
- R46: value 100k -> 1M; Note Base resistor -> Base resistor: 10 uA lights the LED fully
- U10: value LM393 -> LM393B; Note (none) -> The B version (LM393BIDR): output leakage at most 50 nA, wh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
- U9: Note (none) -> OPA1642 has the standard dual op-amp pinout (OPA2134 symbol)
Changed lines of the file:
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@@
 			)
 		)
-		(property "Value" "100pF C0G"
+		(property "Value" "22pF C0G"
 			(at 124.46 167.64 0)
 			(effects
@@
 			)
 		)
-		(property "Note" "RF filter at the op-amp pin"
+		(property "Note" "RF filter at the op-amp pin: 7 MHz with the 1k. Small, because it adds to the guitar lead's capacitance (simulation A1); the OPA1642 rejects GHz RF itself"
 			(at 124.46 165.1 0)
 			(effects
@@
 			)
 		)
-		(property "Datasheet" "http://www.ti.com/lit/ds/symlink/opa134.pdf"
+		(property "Datasheet" "https://www.ti.com/lit/ds/symlink/opa1642.pdf"
 			(at 185.42 149.86 0)
 			(effects
@@
 			)
 		)
+		(property "Note" "OPA1642 has the standard dual op-amp pinout (OPA2134 symbol)"
+			(at 185.42 149.86 0)
+			(effects
+				(font
+					(size 1.27 1.27)
+				)
+				(hide yes)
+			)
+		)
 		(pin "5"
 		)
@@
 			)
 		)
-		(property "Datasheet" "http://www.ti.com/lit/ds/symlink/opa134.pdf"
+		(property "Datasheet" "https://www.ti.com/lit/ds/symlink/opa1642.pdf"
 			(at 224.79 170.18 0)
 			(effects
@@
 			)
 		)
+		(property "Note" "OPA1642 has the standard dual op-amp pinout (OPA2134 symbol)"
+			(at 224.79 170.18 0)
+			(effects
+				(font
+					(size 1.27 1.27)
+				)
+				(hide yes)
+			)
+		)
 		(pin "4"
 		)
@@
 			)
 		)
-		(property "Value" "LM393"
+		(property "Value" "LM393B"
 			(at 116.84 238.76 0)
 			(effects
@@
 			)
 		)
+		(property "Note" "The B version (LM393BIDR): output leakage at most 50 nA, which the 2.2M recharge needs (the plain LM393 allows 1 uA when hot)"
+			(at 110.49 234.95 0)
+			(effects
+				(font
+					(size 1.27 1.27)
+				)
+				(hide yes)
+			)
+		)
 		(pin "1"
 		)
@@
 			)
 		)
-		(property "Value" "LM393"
+		(property "Value" "LM393B"
 			(at 116.84 265.43 0)
 			(effects
@@
 			)
 		)
-		(property "Datasheet" "http://www.ti.com/lit/ds/symlink/lm393.pdf"
+		(property "Datasheet" "https://www.ti.com/lit/ds/symlink/lm393.pdf"
 			(at 110.49 261.62 0)
 			(effects
@@
 			)
 		)
+		(property "Note" "The B version (LM393BIDR): output leakage at most 50 nA, which the 2.2M recharge needs (the plain LM393 allows 1 uA when hot)"
+			(at 110.49 261.62 0)
+			(effects
+				(font
+					(size 1.27 1.27)
+				)
+				(hide yes)
+			)
+		)
 		(pin "5"
 		)
@@
 			)
 		)
-		(property "Value" "LM393"
+		(property "Value" "LM393B"
 			(at 146.05 265.43 0)
 			(effects
@@
 			)
 		)
-		(property "Datasheet" "http://www.ti.com/lit/ds/symlink/lm393.pdf"
+		(property "Datasheet" "https://www.ti.com/lit/ds/symlink/lm393.pdf"
 			(at 139.7 261.62 0)
 			(effects
@@
 			)
 		)
+		(property "Note" "The B version (LM393BIDR): output leakage at most 50 nA, which the 2.2M recharge needs (the plain LM393 allows 1 uA when hot)"
+			(at 139.7 261.62 0)
+			(effects
+				(font
+					(size 1.27 1.27)
+				)
+				(hide yes)
+			)
+		)
 		(pin "4"
 		)
@@
 			)
 		)
-		(property "Note" "Discharges the hold capacitor quickly (about 5 mA)"
+		(property "Note" "Discharges the hold capacitor quickly: 5.5 mA, inside the LM393B's 6 mA minimum sink"
 			(at 170.18 229.87 0)
 			(effects
@@
 			)
 		)
-		(property "Value" "47k"
+		(property "Value" "2.2M"
 			(at 185.42 219.71 90)
 			(effects
@@
 	)
 	(symbol
-		(lib_id "Device:C_Polarized")
+		(lib_id "Device:C")
 		(at 185.42 245.11 0)
 		(unit 1)
@@
 			)
 		)
-		(property "Value" "2.2uF 25V"
+		(property "Value" "100nF"
 			(at 185.42 247.65 0)
 			(effects
@@
 			)
 		)
-		(property "Footprint" "Capacitor_SMD:CP_Elec_4x5.4"
+		(property "Footprint" "Capacitor_SMD:C_0603_1608Metric"
 			(at 186.69 248.92 0)
 			(effects
@@
 			)
 		)
-		(property "Description" "Polarized capacitor"
+		(property "Description" "Unpolarized capacitor"
 			(at 185.42 245.11 0)
 			(effects
@@
 			)
 		)
-		(property "Note" "Hold: LED stays on about 100 ms after a peak (simulation A4)"
+		(property "Note" "Hold: one 1 kHz peak 0.5 dB over the threshold lights the LED for about 100 ms (simulation A4)"
 			(at 185.42 245.11 0)
 			(effects
@@
 			)
 		)
-		(property "Value" "100k"
+		(property "Value" "1M"
 			(at 204.47 234.95 90)
 			(effects
@@
 			)
 		)
-		(property "Note" "Base resistor"
+		(property "Note" "Base resistor: 10 uA lights the LED fully"
 			(at 204.47 234.95 0)
 			(effects

Commit message: Pedalboard PCB: first layout, and Alps RK09L pots
A 4-layer, 208 x 90 mm board, placed and routed from the netlist: the
jacks, knobs, button and clip LED meet the rear panel at the board edge
(from the makers' drawings), small parts sit at the pins the schematic
names, ground plane on In1, routed with Freerouting. Not finished:
4 nets left unrouted, silkscreen to tidy, 3D check to do.

All three knobs are now Alps RK09L12B0A4S (dual 10k log, M9 thread):
the RK09K had no threaded bushing and Alps makes no 50k log single-gang
RK09L. The gain stage's resistors are scaled by 1/5 to keep the same
gain (simulations A1-A3, A5, A7 re-run: pass, noise 1.0 dB). Footprints
from the symbol libraries are kept (14 parts had none), and the MIDI
jack has its own footprint (pedalboard.pretty).

Co-Authored-By: Claude Opus 5.5 <noreply@anthropic.com>
Parts:
- added unit 2 of RV1
- C46: value 47pF C0G -> 220pF C0G
- C47: value 47uF 16V -> 100uF 16V; footprint Capacitor_SMD:CP_Elec_5x5.4 -> Capacitor_SMD:CP_Elec_6.3x5.4
- D4: footprint (none) -> Package_TO_SOT_SMD:SOT-23
- D5: footprint LED_THT:LED_D3.0mm_Horizontal_O1.27mm_Z10.0mm -> LED_THT:LED_D3.0mm_Horizontal_O1.27mm_Z6.0mm
- J5: footprint (none) -> Connector_Audio:Jack_6.35mm_Neutrik_NMJ6HCD2_Horizontal
- R38: value 100k -> 20k; Note Across the pot: Rf at most 33k -> Across the pot: Rf at most 6.7k
- R39: value 2.2k -> 442; Note Rg -> Rg. Low, so it adds little noise: 2.7 nV/rtHz against the o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
- RV1: value 50k gain -> 10k log dual, gain; footprint Potentiometer_THT:Potentiometer_Alps_RK09K_Single_Horizontal -> Potentiometer_THT:Potentiometer_Alps_RK09L_Double_Horizontal; symbol Device:R_Potentiometer -> Device:R_Potentiometer_Dual_Separate; MPN (none) -> Alps RK09L12B0A4S; Note Gain knob, used as a variable resistor: more resistance (ga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 -> Gain knob: one gang used as a variable resistor, terminals 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
Connections:
- net GND: now also RV1.4, RV1.5, RV1.6
Other:
- note added: "Gain stage (5.3): gain = 1 + Rf / 442; Rf = 0 .. 6.7k (pot with 20k across it): 0 .. +24 dB"
- note added: "Spare gang, grounded"
- note removed: "Gain stage (5.3): gain = 1 + Rf / 2.2k; Rf = 0 .. 33k (pot with 100k across it): 0 .. +24 dB"

Commit message: Pedalboard PCB: maker part numbers and LCSC numbers on every part
Each part on the schematic and the board now carries Manufacturer, MPN
and LCSC fields, for the PCBWay and JLCPCB assembly BOMs. FB1 is the
2 A bead (no 0805 bead is rated 3 A), F1 the MF-MSMF150-2 fuse. The
drill/place origin is the board's bottom-left corner, so the Gerbers,
drill and placement files measure from the board.

Co-Authored-By: Claude Opus 5.5 <noreply@anthropic.com>
Parts:
- C40: LCSC (none) -> C72515; MPN (none) -> RVT1C470M0505; Manufacturer (none) -> ROQANG
- C41, C44, C48, C49, C50, C51: LCSC (none) -> C14663; MPN (none) -> CC0603KRX7R9BB104; Manufacturer (none) -> YAGEO
- C42: LCSC (none) -> C97946; MPN (none) -> GRM31C5C1H104JA01L; Manufacturer (none) -> Murata
- C43: LCSC (none) -> C1653; MPN (none) -> CL10C220JB8NNNC; Manufacturer (none) -> Samsung
- C45: LCSC (none) -> C13585; MPN (none) -> CL31A106KBHNNNE; Manufacturer (none) -> Samsung
- C46: LCSC (none) -> C388907; MPN (none) -> GCM1885C2A221JA16D; Manufacturer (none) -> Murata
- C47: LCSC (none) -> C72475; MPN (none) -> RVT1C101M0605; Manufacturer (none) -> ROQANG
- D4: LCSC (none) -> C2500; MPN (none) -> BAV99,215; Manufacturer (none) -> Nexperia
- D5: LCSC (none) -> C99771; MPN (none) -> 204-10SURD/S530-A3-L; Manufacturer (none) -> Everlight
- J5: LCSC (none) -> C368502; MPN (none) -> NMJ6HCD2; Manufacturer (none) -> Neutrik
- Q1: LCSC (none) -> C8666; MPN (none) -> BC857C,215; Manufacturer (none) -> Nexperia
- R33: LCSC (none) -> C185372; MPN (none) -> RC0603FR-07140KL; Manufacturer (none) -> YAGEO
- R34: LCSC (none) -> C25803; MPN (none) -> 0603WAF1003T5E; Manufacturer (none) -> UNI-ROYAL
- R35: LCSC (none) -> C7250; MPN (none) -> 0603WAF1005T5E; Manufacturer (none) -> UNI-ROYAL
- R36: LCSC (none) -> C21190; MPN (none) -> 0603WAF1001T5E; Manufacturer (none) -> UNI-ROYAL
- R37, R46: LCSC (none) -> C22935; MPN (none) -> 0603WAF1004T5E; Manufacturer (none) -> UNI-ROYAL
- R38: LCSC (none) -> C4184; MPN (none) -> 0603WAF2002T5E; Manufacturer (none) -> UNI-ROYAL
- R39: LCSC (none) -> C23057; MPN (none) -> 0603WAF4420T5E; Manufacturer (none) -> UNI-ROYAL
- R40: LCSC (none) -> C855860; MPN (none) -> AT0603BRD0744K2L; Manufacturer (none) -> YAGEO
- R41: LCSC (none) -> C304764; MPN (none) -> RS-03K5232FT; Manufacturer (none) -> FH
- R42: LCSC (none) -> C136968; MPN (none) -> RT0603BRD0724K3L; Manufacturer (none) -> YAGEO
- R43: LCSC (none) -> C25804; MPN (none) -> 0603WAF1002T5E; Manufacturer (none) -> UNI-ROYAL
- R44: LCSC (none) -> C4190; MPN (none) -> 0603WAF2201T5E; Manufacturer (none) -> UNI-ROYAL
- R45: LCSC (none) -> C22938; MPN (none) -> 0603WAF2204T5E; Manufacturer (none) -> UNI-ROYAL
- R47: LCSC (none) -> C23162; MPN (none) -> 0603WAF4701T5E; Manufacturer (none) -> UNI-ROYAL
- RV1: MPN Alps RK09L12B0A4S -> RK09L12B0A4S; Manufacturer (none) -> Alps Alpine
- U10: MPN (none) -> LM393BIDR; Manufacturer (none) -> Texas Instruments
- U9: LCSC (none) -> C67640; MPN (none) -> OPA1642AIDR; Manufacturer (none) -> Texas Instruments
