File: pcb/kicad/outputs.kicad_sch (KiCad schematic)
At the start: 33 parts, among them J6 Main out L, J7 Main out R, J8 Headphones, U11 OPA1642AIDR, U12 TPA6130A2RTJR

Commit message: Pedalboard PCB: simulations A1-A8 and the values they changed
ngspice simulations of the guitar input, clip LED, ADC input, outputs,
headphones and the 12 V supply, read from the KiCad netlist and run with
TI's models (fetched by get-models.sh, not in git). All eight pass.

From the simulations: guitar RF filter 100 pF -> 22 pF, clip LED hold
100 nF / 2.2M / 1M with the LM393B, main output capacitors 47 uF.
The power-off thump when the lead is pulled is accepted for now
(sim/README.md).

Co-Authored-By: Claude Opus 5.5 <noreply@anthropic.com>
Parts:
- C53, C55: value 10uF 25V -> 47uF 25V; footprint Capacitor_SMD:CP_Elec_5x5.4 -> Capacitor_SMD:CP_Elec_6.3x5.4; Note + toward the buffer (5 V) -> + toward the buffer (5 V). 47 uF: -3 dB at 4 Hz into 600 oh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
- U11: Note (none) -> Unity-gain buffer
Other:
- note added: "Main outputs (5.5): DAC -> volume -> buffer -> 47 uF -> 100 ohm -> tip; ring -> 100 ohm -> ground"
- note removed: "Main outputs (5.5): DAC -> volume -> buffer -> 10 uF -> 100 ohm -> tip; ring -> 100 ohm -> ground"
Changed lines of the file:
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@@
 		)
 	)
-	(text "Main outputs (5.5): DAC -> volume -> buffer -> 10 uF -> 100 ohm -> tip; ring -> 100 ohm -> ground"
+	(text "Main outputs (5.5): DAC -> volume -> buffer -> 47 uF -> 100 ohm -> tip; ring -> 100 ohm -> ground"
 		(exclude_from_sim no)
 		(at 20 48 0)
@@
 			)
 		)
-		(property "Value" "10uF 25V"
+		(property "Value" "47uF 25V"
 			(at 154.94 82.55 0)
 			(effects
@@
 			)
 		)
-		(property "Footprint" "Capacitor_SMD:CP_Elec_5x5.4"
+		(property "Footprint" "Capacitor_SMD:CP_Elec_6.3x5.4"
 			(at 156.21 83.82 0)
 			(effects
@@
 			)
 		)
-		(property "Note" "+ toward the buffer (5 V)"
+		(property "Note" "+ toward the buffer (5 V). 47 uF: -3 dB at 4 Hz into 600 ohm (10 uF gave 20 Hz, simulation A6)"
 			(at 154.94 80.01 0)
 			(effects
@@
 			)
 		)
-		(property "Value" "10uF 25V"
+		(property "Value" "47uF 25V"
 			(at 154.94 127 0)
 			(effects
@@
 			)
 		)
-		(property "Footprint" "Capacitor_SMD:CP_Elec_5x5.4"
+		(property "Footprint" "Capacitor_SMD:CP_Elec_6.3x5.4"
 			(at 156.21 128.27 0)
 			(effects
@@
 			)
 		)
-		(property "Note" "+ toward the buffer (5 V)"
+		(property "Note" "+ toward the buffer (5 V). 47 uF: -3 dB at 4 Hz into 600 ohm (10 uF gave 20 Hz, simulation A6)"
 			(at 154.94 124.46 0)
 			(effects
@@
 			)
 		)
-		(property "Datasheet" "http://www.ti.com/lit/ds/symlink/opa134.pdf"
+		(property "Datasheet" "https://www.ti.com/lit/ds/symlink/opa1642.pdf"
 			(at 124.46 160.02 0)
 			(effects
@@
 			(at 124.46 160.02 0)
 			(effects
+				(font
+					(size 1.27 1.27)
+				)
+				(hide yes)
+			)
+		)
+		(property "Note" "Unity-gain buffer"
+			(at 124.46 160.02 0)
+			(effects

Commit message: Pedalboard PCB: first layout, and Alps RK09L pots
A 4-layer, 208 x 90 mm board, placed and routed from the netlist: the
jacks, knobs, button and clip LED meet the rear panel at the board edge
(from the makers' drawings), small parts sit at the pins the schematic
names, ground plane on In1, routed with Freerouting. Not finished:
4 nets left unrouted, silkscreen to tidy, 3D check to do.

All three knobs are now Alps RK09L12B0A4S (dual 10k log, M9 thread):
the RK09K had no threaded bushing and Alps makes no 50k log single-gang
RK09L. The gain stage's resistors are scaled by 1/5 to keep the same
gain (simulations A1-A3, A5, A7 re-run: pass, noise 1.0 dB). Footprints
from the symbol libraries are kept (14 parts had none), and the MIDI
jack has its own footprint (pedalboard.pretty).

Co-Authored-By: Claude Opus 5.5 <noreply@anthropic.com>
Parts:
- J6, J7, J8: footprint (none) -> Connector_Audio:Jack_6.35mm_Neutrik_NMJ6HCD2_Horizontal
- RV2, RV3: MPN (none) -> Alps RK09L12B0A4S
- U12: footprint (none) -> Package_DFN_QFN:QFN-20-1EP_4x4mm_P0.5mm_EP2.7x2.7mm
Changed lines of the file:
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@@
 			)
 		)
-		(property "Datasheet" "~"
+		(property "Datasheet" "https://tech.alpsalpine.com/e/products/detail/RK09L12B0A4S/"
 			(at 54.61 80.01 0)
 			(effects
@@
 			)
 		)
+		(property "MPN" "Alps RK09L12B0A4S"
+			(at 54.61 80.01 0)
+			(effects
+				(font
+					(size 1.27 1.27)
+				)
+				(hide yes)
+			)
+		)
 		(pin "1"
 		)
@@
 			)
 		)
-		(property "Datasheet" "~"
+		(property "Datasheet" "https://tech.alpsalpine.com/e/products/detail/RK09L12B0A4S/"
 			(at 54.61 124.46 0)
 			(effects
@@
 			)
 		)
+		(property "MPN" "Alps RK09L12B0A4S"
+			(at 54.61 124.46 0)
+			(effects
+				(font
+					(size 1.27 1.27)
+				)
+				(hide yes)
+			)
+		)
 		(pin "4"
 		)
@@
 			)
 		)
-		(property "Footprint" ""
+		(property "Footprint" "Connector_Audio:Jack_6.35mm_Neutrik_NMJ6HCD2_Horizontal"
 			(at 224.79 80.01 0)
 			(effects
@@
 			)
 		)
-		(property "Footprint" ""
+		(property "Footprint" "Connector_Audio:Jack_6.35mm_Neutrik_NMJ6HCD2_Horizontal"
 			(at 224.79 124.46 0)
 			(effects
@@
 			)
 		)
-		(property "Datasheet" "~"
+		(property "Datasheet" "https://tech.alpsalpine.com/e/products/detail/RK09L12B0A4S/"
 			(at 59.69 214.63 0)
 			(effects
@@
 			)
 		)
+		(property "MPN" "Alps RK09L12B0A4S"
+			(at 59.69 214.63 0)
+			(effects
+				(font
+					(size 1.27 1.27)
+				)
+				(hide yes)
+			)
+		)
 		(pin "1"
 		)
@@
 			)
 		)
-		(property "Datasheet" "~"
+		(property "Datasheet" "https://tech.alpsalpine.com/e/products/detail/RK09L12B0A4S/"
 			(at 59.69 245.11 0)
 			(effects
@@
 			)
 		)
+		(property "MPN" "Alps RK09L12B0A4S"
+			(at 59.69 245.11 0)
+			(effects
+				(font
+					(size 1.27 1.27)
+				)
+				(hide yes)
+			)
+		)
 		(pin "4"
 		)
@@
 			)
 		)
-		(property "Footprint" ""
+		(property "Footprint" "Package_DFN_QFN:QFN-20-1EP_4x4mm_P0.5mm_EP2.7x2.7mm"
 			(at 160.02 234.95 0)
 			(effects
@@
 			)
 		)
-		(property "Footprint" ""
+		(property "Footprint" "Connector_Audio:Jack_6.35mm_Neutrik_NMJ6HCD2_Horizontal"
 			(at 250.19 229.87 0)
 			(effects

Commit message: Pedalboard PCB: maker part numbers and LCSC numbers on every part
Each part on the schematic and the board now carries Manufacturer, MPN
and LCSC fields, for the PCBWay and JLCPCB assembly BOMs. FB1 is the
2 A bead (no 0805 bead is rated 3 A), F1 the MF-MSMF150-2 fuse. The
drill/place origin is the board's bottom-left corner, so the Gerbers,
drill and placement files measure from the board.

Co-Authored-By: Claude Opus 5.5 <noreply@anthropic.com>
Parts:
- C52, C54: LCSC (none) -> C72511; MPN (none) -> RVT1V4R7M0405; Manufacturer (none) -> ROQANG
- C53, C55: LCSC (none) -> C72521; MPN (none) -> RVT1E470M0605; Manufacturer (none) -> ROQANG
- C56: LCSC (none) -> C14663; MPN (none) -> CC0603KRX7R9BB104; Manufacturer (none) -> YAGEO
- C57: LCSC (none) -> C13585; MPN (none) -> CL31A106KBHNNNE; Manufacturer (none) -> Samsung
- C58, C59, C60, C61: LCSC (none) -> C13967; MPN (none) -> CL21B474KBFNNNE; Manufacturer (none) -> Samsung
- C62, C63, C65, C66: LCSC (none) -> C15849; MPN (none) -> CL10A105KB8NNNC; Manufacturer (none) -> Samsung
- C64: LCSC (none) -> C15850; MPN (none) -> CL21A106KAYNNNE; Manufacturer (none) -> Samsung
- J6, J7, J8: LCSC (none) -> C368502; MPN (none) -> NMJ6HCD2; Manufacturer (none) -> Neutrik
- R48, R49, R52, R53: LCSC (none) -> C25803; MPN (none) -> 0603WAF1003T5E; Manufacturer (none) -> UNI-ROYAL
- R50, R51, R54, R55: LCSC (none) -> C22775; MPN (none) -> 0603WAF1000T5E; Manufacturer (none) -> UNI-ROYAL
- R56, R57, R58: LCSC (none) -> C25804; MPN (none) -> 0603WAF1002T5E; Manufacturer (none) -> UNI-ROYAL
- RV2, RV3: MPN Alps RK09L12B0A4S -> RK09L12B0A4S; Manufacturer (none) -> Alps Alpine
- U11: LCSC (none) -> C67640; MPN (none) -> OPA1642AIDR; Manufacturer (none) -> Texas Instruments
- U12: LCSC (none) -> C130046; MPN (none) -> TPA6130A2RTJR; Manufacturer (none) -> Texas Instruments
