File: pcb/kicad/pico.kicad_sch (KiCad schematic)
At the start: 48 parts, among them J10 Switch 2, J11 Switch 3, J12 Switch 4, J13 Switch 5, J14 Switch 6, J15 Switch 7, J16 Switch 8, J17 Expression, J18 MIDI out, J9 Switch 1, U13 SRV05-4, U14 SRV05-4, U15 SRV05-4, U16 SRV05-4, U17 SRV05-4

Commit message: Pedalboard PCB: first layout, and Alps RK09L pots
A 4-layer, 208 x 90 mm board, placed and routed from the netlist: the
jacks, knobs, button and clip LED meet the rear panel at the board edge
(from the makers' drawings), small parts sit at the pins the schematic
names, ground plane on In1, routed with Freerouting. Not finished:
4 nets left unrouted, silkscreen to tidy, 3D check to do.

All three knobs are now Alps RK09L12B0A4S (dual 10k log, M9 thread):
the RK09K had no threaded bushing and Alps makes no 50k log single-gang
RK09L. The gain stage's resistors are scaled by 1/5 to keep the same
gain (simulations A1-A3, A5, A7 re-run: pass, noise 1.0 dB). Footprints
from the symbol libraries are kept (14 parts had none), and the MIDI
jack has its own footprint (pedalboard.pretty).

Co-Authored-By: Claude Opus 5.5 <noreply@anthropic.com>
Parts:
- J17: footprint (none) -> Connector_Audio:Jack_6.35mm_Neutrik_NMJ6HCD2_Horizontal
- J18: footprint (none) -> pedalboard:Jack_3.5mm_SameSky_SJ1-3543_Horizontal; Note Right-angle 3.5 mm TRS, M6 thread and nut. Footprint drawn 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 -> Right-angle 3.5 mm TRS, M6 thread and nut. Footprint from i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
- JP1, JP2: now left out of the parts list
Changed lines of the file:
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@@
 			)
 		)
-		(property "Footprint" ""
+		(property "Footprint" "Connector_Audio:Jack_6.35mm_Neutrik_NMJ6HCD2_Horizontal"
 			(at 30.48 209.55 0)
 			(effects
@@
 		(unit 1)
 		(exclude_from_sim no)
-		(in_bom yes)
+		(in_bom no)
 		(on_board yes)
 		(dnp no)
@@
 		(unit 1)
 		(exclude_from_sim no)
-		(in_bom yes)
+		(in_bom no)
 		(on_board yes)
 		(dnp no)
@@
 			)
 		)
-		(property "Footprint" ""
+		(property "Footprint" "pedalboard:Jack_3.5mm_SameSky_SJ1-3543_Horizontal"
 			(at 30.48 261.62 0)
 			(effects
@@
 			)
 		)
-		(property "Note" "Right-angle 3.5 mm TRS, M6 thread and nut. Footprint drawn at layout from its datasheet (pads named T, R, S: 2 = tip, 3 = ring, 1 = sleeve)"
+		(property "Note" "Right-angle 3.5 mm TRS, M6 thread and nut. Footprint from its datasheet (gen/mkfp.py; pads named T, R, S: 2 = tip, 3 = ring, 1 = sleeve)"
 			(at 30.48 261.62 0)
 			(effects

Commit message: Pedalboard PCB: maker part numbers and LCSC numbers on every part
Each part on the schematic and the board now carries Manufacturer, MPN
and LCSC fields, for the PCBWay and JLCPCB assembly BOMs. FB1 is the
2 A bead (no 0805 bead is rated 3 A), F1 the MF-MSMF150-2 fuse. The
drill/place origin is the board's bottom-left corner, so the Gerbers,
drill and placement files measure from the board.

Co-Authored-By: Claude Opus 5.5 <noreply@anthropic.com>
Parts:
- A1: MPN (none) -> Pico H; Manufacturer (none) -> Raspberry Pi
- C67, C68, C69, C70, C71, C72, C73, C74, C75: LCSC (none) -> C57112; MPN (none) -> 0603B103K500NT; Manufacturer (none) -> FH
- J10, J11, J12, J13, J14, J15, J16, J9: LCSC (none) -> C144395; MPN (none) -> B4B-XH-A(LF)(SN); Manufacturer (none) -> JST
- J17: LCSC (none) -> C368502; MPN (none) -> NMJ6HCD2; Manufacturer (none) -> Neutrik
- J18: MPN Same Sky SJ1-3543 -> SJ1-3543; Manufacturer (none) -> Same Sky
- R59, R61, R63, R65, R67, R69, R71, R73, R75, R77: LCSC (none) -> C21190; MPN (none) -> 0603WAF1001T5E; Manufacturer (none) -> UNI-ROYAL
- R60, R62, R64, R66, R68, R70, R72, R74: LCSC (none) -> C23179; MPN (none) -> 0603WAF4700T5E; Manufacturer (none) -> UNI-ROYAL
- R76: LCSC (none) -> C22935; MPN (none) -> 0603WAF1004T5E; Manufacturer (none) -> UNI-ROYAL
- R78: LCSC (none) -> C22859; MPN (none) -> 0603WAF100JT5E; Manufacturer (none) -> UNI-ROYAL
- R79: LCSC (none) -> C723447; MPN (none) -> RC1210FR-0733RL; Manufacturer (none) -> YAGEO
- U13, U14, U15, U16, U17: LCSC (none) -> C384887; MPN (none) -> SRV05-4; Manufacturer (none) -> Leiditech
