File: pcb/kicad/power.kicad_sch (KiCad schematic)
At the start: 40 parts, among them U1 TLV75733PDBV, U2 TPS7A2033PDBV, U3 TPS61040DBV, U4 TPS7A4901DGN

Commit message: Pedalboard PCB: audio converters and clocks sheet
PCM5122 DAC (0x4D, clock master) and PCM1863 ADC (0x4A), wired as the
HiFiBerry DAC+ADC Pro driver expects; Kyocera 22.5792 and 24.576 MHz
oscillators enabled by the DAC's GPIO6/GPIO3 and joined by an OR gate;
DAC output filters and the ADC's input filter from TI's datasheets.

Co-Authored-By: Claude Opus 5.5 <noreply@anthropic.com>
Changed lines of the file:
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@@
 		(pts
 			(xy 113.03 242.57)
-			(xy 113.03 245.11)
+			(xy 113.03 250.19)
 		)
 		(stroke
@@
 	(symbol
 		(lib_id "power:GND")
-		(at 113.03 245.11 0)
+		(at 113.03 250.19 0)
 		(unit 1)
 		(exclude_from_sim no)
@@
 		(dnp no)
 		(property "Reference" "#PWR054"
-			(at 113.03 251.46 0)
+			(at 113.03 256.54 0)
 			(effects
 				(font
@@
 		)
 		(property "Value" "GND"
-			(at 113.03 248.92 0)
+			(at 113.03 254 0)
 			(effects
 				(font
@@
 		)
 		(property "Footprint" ""
-			(at 113.03 245.11 0)
+			(at 113.03 250.19 0)
 			(effects
 				(font
@@
 		)
 		(property "Datasheet" ""
-			(at 113.03 245.11 0)
+			(at 113.03 250.19 0)
 			(effects
 				(font
@@
 		)
 		(property "Description" "Power symbol creates a global label with name \"GND\" , ground"
-			(at 113.03 245.11 0)
+			(at 113.03 250.19 0)
 			(effects
 				(font

Commit message: Pedalboard PCB: first layout, and Alps RK09L pots
A 4-layer, 208 x 90 mm board, placed and routed from the netlist: the
jacks, knobs, button and clip LED meet the rear panel at the board edge
(from the makers' drawings), small parts sit at the pins the schematic
names, ground plane on In1, routed with Freerouting. Not finished:
4 nets left unrouted, silkscreen to tidy, 3D check to do.

All three knobs are now Alps RK09L12B0A4S (dual 10k log, M9 thread):
the RK09K had no threaded bushing and Alps makes no 50k log single-gang
RK09L. The gain stage's resistors are scaled by 1/5 to keep the same
gain (simulations A1-A3, A5, A7 re-run: pass, noise 1.0 dB). Footprints
from the symbol libraries are kept (14 parts had none), and the MIDI
jack has its own footprint (pedalboard.pretty).

Co-Authored-By: Claude Opus 5.5 <noreply@anthropic.com>
Parts:
- TP1, TP2, TP3, TP4, TP5, TP6, TP7: now left out of the parts list
- U1, U2, U3: footprint (none) -> Package_TO_SOT_SMD:SOT-23-5
- U4: footprint (none) -> Package_SO:HVSSOP-8-1EP_3x3mm_P0.65mm_EP1.57x1.89mm
Changed lines of the file:
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@@
 		(unit 1)
 		(exclude_from_sim no)
-		(in_bom yes)
+		(in_bom no)
 		(on_board yes)
 		(dnp no)
@@
 		(unit 1)
 		(exclude_from_sim no)
-		(in_bom yes)
+		(in_bom no)
 		(on_board yes)
 		(dnp no)
@@
 		(unit 1)
 		(exclude_from_sim no)
-		(in_bom yes)
+		(in_bom no)
 		(on_board yes)
 		(dnp no)
@@
 			)
 		)
-		(property "Footprint" ""
+		(property "Footprint" "Package_TO_SOT_SMD:SOT-23-5"
 			(at 54.61 101.6 0)
 			(effects
@@
 		(unit 1)
 		(exclude_from_sim no)
-		(in_bom yes)
+		(in_bom no)
 		(on_board yes)
 		(dnp no)
@@
 			)
 		)
-		(property "Footprint" ""
+		(property "Footprint" "Package_TO_SOT_SMD:SOT-23-5"
 			(at 204.47 110.49 0)
 			(effects
@@
 		(unit 1)
 		(exclude_from_sim no)
-		(in_bom yes)
+		(in_bom no)
 		(on_board yes)
 		(dnp no)
@@
 			)
 		)
-		(property "Footprint" ""
+		(property "Footprint" "Package_TO_SOT_SMD:SOT-23-5"
 			(at 77.47 171.45 0)
 			(effects
@@
 		(unit 1)
 		(exclude_from_sim no)
-		(in_bom yes)
+		(in_bom no)
 		(on_board yes)
 		(dnp no)
@@
 			)
 		)
-		(property "Footprint" ""
+		(property "Footprint" "Package_SO:HVSSOP-8-1EP_3x3mm_P0.65mm_EP1.57x1.89mm"
 			(at 110.49 228.6 0)
 			(effects
@@
 		(unit 1)
 		(exclude_from_sim no)
-		(in_bom yes)
+		(in_bom no)
 		(on_board yes)
 		(dnp no)

Commit message: Pedalboard PCB: maker part numbers and LCSC numbers on every part
Each part on the schematic and the board now carries Manufacturer, MPN
and LCSC fields, for the PCBWay and JLCPCB assembly BOMs. FB1 is the
2 A bead (no 0805 bead is rated 3 A), F1 the MF-MSMF150-2 fuse. The
drill/place origin is the board's bottom-left corner, so the Gerbers,
drill and placement files measure from the board.

Co-Authored-By: Claude Opus 5.5 <noreply@anthropic.com>
Parts:
- C1: LCSC (none) -> C12891; MPN (none) -> CL31A226KAHNNNE; Manufacturer (none) -> Samsung
- C10: LCSC (none) -> C170099; MPN (none) -> CL32B475KBUYNNE; Manufacturer (none) -> Samsung
- C11, C14: LCSC (none) -> C13585; MPN (none) -> CL31A106KBHNNNE; Manufacturer (none) -> Samsung
- C12, C13: LCSC (none) -> C57112; MPN (none) -> 0603B103K500NT; Manufacturer (none) -> FH
- C2: LCSC (none) -> C14663; MPN (none) -> CC0603KRX7R9BB104; Manufacturer (none) -> YAGEO
- C3, C4, C6, C7: LCSC (none) -> C15849; MPN (none) -> CL10A105KB8NNNC; Manufacturer (none) -> Samsung
- C5: LCSC (none) -> C15850; MPN (none) -> CL21A106KAYNNNE; Manufacturer (none) -> Samsung
- C8: LCSC (none) -> C1779; MPN (none) -> CL21A475KAQNNNE; Manufacturer (none) -> Samsung
- C9: LCSC (none) -> C1653; MPN (none) -> CL10C220JB8NNNC; Manufacturer (none) -> Samsung
- D1: LCSC (none) -> C82046; MPN (none) -> MBR0530T1G; Manufacturer (none) -> onsemi
- F1: LCSC (none) -> C89648; MPN (none) -> MF-MSMF150-2; Manufacturer (none) -> Bourns; Note PTC, ~1.5 A hold, under 0.1 V drop at 1 A (plan C3) -> PTC, 1.5 A hold, 3 A trip; 30 mohm new, 0.12 ohm at most af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
- FB1: value 220R@100MHz 3A -> 220R@100MHz 2A; LCSC (none) -> C85840; MPN (none) -> BLM21PG221SN1D; Manufacturer (none) -> Murata; Note Rated 3 A, DC resistance under 0.05 ohm -> Rated 2 A (the board draws 1.2 A at most), 45 mohm (no 0805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
- FB2: LCSC (none) -> C85833; MPN (none) -> BLM18KG601SN1D; Manufacturer (none) -> Murata
- L1: LCSC (none) -> C98020; MPN (none) -> LQH32PN100MN0L; Manufacturer (none) -> Murata
- R1: LCSC (none) -> C21190; MPN (none) -> 0603WAF1001T5E; Manufacturer (none) -> UNI-ROYAL
- R10, R3, R4: LCSC (none) -> C21189; MPN (none) -> 0603WAF0000T5E; Manufacturer (none) -> UNI-ROYAL
- R2, R9: LCSC (none) -> C25803; MPN (none) -> 0603WAF1003T5E; Manufacturer (none) -> UNI-ROYAL
- R5: LCSC (none) -> C59295; MPN (none) -> 0603WAF1784T5E; Manufacturer (none) -> UNI-ROYAL
- R6: LCSC (none) -> C22813; MPN (none) -> 0603WAF1603T5E; Manufacturer (none) -> UNI-ROYAL
- R7: LCSC (none) -> C26010; MPN (none) -> 0805W8F3301T5E; Manufacturer (none) -> UNI-ROYAL
- R8: LCSC (none) -> C138276; MPN (none) -> AC0603FR-07909KL; Manufacturer (none) -> YAGEO
- U1: LCSC (none) -> C485517; MPN (none) -> TLV75733PDBVR; Manufacturer (none) -> Texas Instruments
- U2: MPN (none) -> TPS7A2033PDBVR; Manufacturer (none) -> Texas Instruments
- U3: LCSC (none) -> C7722; MPN (none) -> TPS61040DBVR; Manufacturer (none) -> Texas Instruments
- U4: LCSC (none) -> C16430; MPN (none) -> TPS7A4901DGNR; Manufacturer (none) -> Texas Instruments
